Commit message: Update rslidar_2d.urdf

File: rslidar_2d.urdf (robot description, URDF)
Before this commit: robot myrobot_udrf, 17 links, 16 joints
Joints:
- joint imu_link_joint: origin xyz=-0.023 0 0.4 rpy=0 0 0 -> xyz=-0.023 0 0.4 rpy=0 0 3.14159

Commit message: Update rslidar_2d.urdf

File: rslidar_2d.urdf (robot description, URDF)
Before this commit: robot myrobot_udrf, 17 links, 16 joints
Links:
- added link base_footprint
- link base_link: geometry visual box size=0.415 .4284 .15
- link middle_link: geometry visual box size=0.415 .4284 .001
- link top_link: geometry visual box size=0.2142 .415 .001
Joints:
- added joint base_link_joint: type fixed, parent base_footprint, child base_link, origin xyz=0 0 0.117635
- joint horizontal_laser_link_joint: origin xyz=0 -0.07 0.466 rpy=0 0 0 -> xyz=-0.07 0 0.04135 rpy=0 0 0; parent base_link -> top_link
- joint imu_link_joint: origin xyz=-0.023 0 0.4 rpy=0 0 3.14159 -> xyz=0 0.023 0.02 rpy=0 0 3.14159; parent base_link -> middle_link
- joint left_back_wheel_joint: origin xyz=-0.2142 -0.205 -0.06 rpy=0 1.57075 0 -> xyz=-0.205 0.2142 -0.06 rpy=1.57075 0 0
- joint left_front_wheel_joint: origin xyz=-0.2142 0.205 -0.06 rpy=0 1.57075 0 -> xyz=0.205 .2142 -0.06 rpy=1.57075 0 0
- joint pillar_left_back_joint: origin xyz=-0.15 -0.15 0.19 rpy=0 0 0 -> xyz=-0.15 0.15 0.19 rpy=0 0 0
- joint pillar_left_front_joint: origin xyz=-0.15 0.15 0.19 rpy=0 0 0 -> xyz=0.15 0.15 0.19 rpy=0 0 0
- joint pillar_right_back_joint: origin xyz=0.15 -0.15 0.19 rpy=0 0 0 -> xyz=-0.15 -0.15 0.19 rpy=0 0 0
- joint pillar_right_front_joint: origin xyz=0.15 0.15 0.19 rpy=0 0 0 -> xyz=0.15 -0.15 0.19 rpy=0 0 0
- joint right_back_wheel_joint: origin xyz=0.2142 -0.205 -0.06 rpy=0 1.57075 0 -> xyz=-0.205 -0.2142 -0.06 rpy=1.57075 0 0
- joint right_front_wheel_joint: origin xyz=0.2142 0.205 -0.06 rpy=0 1.57075 0 -> xyz=0.205 -0.2142 -0.06 rpy=1.57075 0 0
- joint top_link_joint: origin xyz=0 -0.07 0.04465 rpy=0 0 0 -> xyz=-0.07 0 0.04465 rpy=0 0 0
- joint top_pillar_left_back_joint: origin xyz=-0.1 -0.1 0.022 rpy=0 0 0 -> xyz=-0.1 0.1 0.022 rpy=0 0 0
- joint top_pillar_left_front_joint: origin xyz=-0.1 -0.04 0.022 rpy=0 0 0 -> xyz=-0.04 0.1 0.022 rpy=0 0 0
- joint top_pillar_right_back_joint: origin xyz=0.1 -0.1 0.022 rpy=0 0 0 -> xyz=-0.1 -0.1 0.022 rpy=0 0 0
- joint top_pillar_right_front_joint: origin xyz=0.1 -0.04 0.022 rpy=0 0 0 -> xyz=-0.04 -0.1 0.022 rpy=0 0 0

Commit message: Update rslidar_2d.urdf

File: rslidar_2d.urdf (robot description, URDF)
Before this commit: robot myrobot_udrf, 18 links, 17 joints
Joints:
- joint horizontal_laser_link_joint: origin xyz=-0.07 0 0.04135 rpy=0 0 0 -> xyz=-0.07 0 0.466 rpy=0 0 0; parent top_link -> base_link
- joint imu_link_joint: origin xyz=0 0.023 0.02 rpy=0 0 3.14159 -> xyz=0 0.023 0.4 rpy=0 0 -1.57075; parent middle_link -> base_link
